File: electrolyte.kicad_pcb (KiCad board)
At the start: 2 copper layers, 190.5 x 76.2 mm, 86 parts, among them U1 ProMicro

Commit message: create a modified repo
Parts:
- added MX16_2: MX-NoLED, Button_Switch_Keyboard:SW_Cherry_MX_2.00u_PCB, F.Cu at (90.1, 87.9)
- added MX28_2: MX-NoLED, Button_Switch_Keyboard:SW_Cherry_MX_2.00u_PCB, F.Cu at (128.2, 87.9)
- added SW_RST1: SW_Push, Button_Switch_SMD:SW_SPST_TL3342, B.Cu at (58.7, 35.1)
- moved D16 16.2 mm to (75.0, 83.0)
- moved D24 16.2 mm to (113.1, 83.0)
- turned MX20 to 180 degrees
- turned MX28 to 180 degrees
- turned MX5 to 180 degrees
Connections:
- U1 pad 1: Net-(U1-Pad1) -> unconnected-(U1-Pad1)
- U1 pad 2: Net-(U1-Pad2) -> unconnected-(U1-Pad2)
- U1 pad 21: Net-(U1-Pad21) -> unconnected-(U1-Pad21)
- U1 pad 22: Net-(U1-Pad22) -> RST
- U1 pad 23: Net-(U1-Pad23) -> GND
- U1 pad 24: Net-(U1-Pad24) -> unconnected-(U1-Pad24)
- U1 pad 3: Net-(U1-Pad3) -> GND
- U1 pad 4: Net-(U1-Pad4) -> GND
- U1 pad 5: Net-(U1-Pad5) -> unconnected-(U1-Pad5)
- U1 pad 6: Net-(U1-Pad6) -> unconnected-(U1-Pad6)
Routing:
- net COL4: track 110.8 -> 154.7 mm, vias 0 -> 1
- net COL5: track 129.0 -> 156.3 mm, vias 0 -> 1
- net RST: track 0.00 -> 22.3 mm
- net COL3: track 89.7 -> 111.2 mm, vias 0 -> 1
- net COL6: track 144.4 -> 164.6 mm, vias 0 -> 1
- net Net-(D24-Pad2): track 7.41 -> 26.5 mm
- net Net-(D20-Pad2): track 6.13 -> 24.0 mm
- net GND: track 0.00 -> 17.0 mm, vias 0 -> 13
- net Net-(D5-Pad2): track 9.86 -> 22.1 mm
- net COL7: track 162.8 -> 174.7 mm, vias 0 -> 1
- net COL0: track 74.4 -> 86.2 mm
- net COL8: track 181.4 -> 192.0 mm, vias 0 -> 1
- net Net-(D28-Pad2): track 6.13 -> 15.4 mm
- net ROW3: track 200.3 -> 207.3 mm
- net Net-(D16-Pad2): track 6.13 -> 11.2 mm
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- added copper zone on B.Cu, net GND
- added copper zone on F.Cu, net GND
Other:
- net class Default removed
- board text added: "Designed by rlbaxter Modified by Routa Keebs"
- board text added: "Electrolyte v1.fun"
- board text added: "JLCJLCJLCJLC"
- board text removed: "Designed by rlbaxter"
- board text removed: "Electrolyte v1"
